Commit message: feat: add the perception and task manager

File: src/ros2_rm_robot/rm_description/urdf/rm_65.urdf.xacro (robot description, xacro)
@@ -545,11 +545,11 @@
     </inertial>
     <visual>
-      <origin xyz="0 0 0.125" rpy="0 0 0" />
-      <geometry><cylinder radius="0.005" length="0.25" /></geometry>
+      <origin xyz="0 0 0.246" rpy="0 0 0" />
+      <geometry><cylinder radius="0.005" length="0.492" /></geometry>
       <material name="SurgicalToolSilver"><color rgba="0.78 0.80 0.84 1" /></material>
     </visual>
     <collision>
-      <origin xyz="0 0 0.125" rpy="0 0 0" />
-      <geometry><cylinder radius="0.005" length="0.25" /></geometry>
+      <origin xyz="0 0 0.246" rpy="0 0 0" />
+      <geometry><cylinder radius="0.005" length="0.492" /></geometry>
     </collision>
   </link>
@@ -561,5 +561,5 @@
   <link name="SurgicalToolTip" />
   <joint name="surgical_tool_tip_joint" type="fixed">
-    <origin xyz="0 0 0.25" rpy="0 0 0" />
+    <origin xyz="0 0 0.492" rpy="0 0 0" />
     <parent link="SurgicalTool" />
     <child link="SurgicalToolTip" />

File: src/ros2_rm_robot/rm_description/urdf/rm_65_gazebo.urdf.xacro (robot description, xacro)
@@ -523,11 +523,11 @@
     </inertial>
     <visual>
-      <origin xyz="0 0 0.125" rpy="0 0 0" />
-      <geometry><cylinder radius="0.005" length="0.25" /></geometry>
+      <origin xyz="0 0 0.246" rpy="0 0 0" />
+      <geometry><cylinder radius="0.005" length="0.492" /></geometry>
       <material name="SurgicalToolSilver"><color rgba="0.78 0.80 0.84 1" /></material>
     </visual>
     <collision>
-      <origin xyz="0 0 0.125" rpy="0 0 0" />
-      <geometry><cylinder radius="0.005" length="0.25" /></geometry>
+      <origin xyz="0 0 0.246" rpy="0 0 0" />
+      <geometry><cylinder radius="0.005" length="0.492" /></geometry>
     </collision>
   </link>
@@ -539,5 +539,5 @@
   <link name="SurgicalToolTip" />
   <joint name="surgical_tool_tip_joint" type="fixed">
-    <origin xyz="0 0 0.25" rpy="0 0 0" />
+    <origin xyz="0 0 0.492" rpy="0 0 0" />
     <parent link="SurgicalTool" />
     <child link="SurgicalToolTip" />

File: src/ros2_rm_robot/rm_moveit2_config/rm_65_config/config/rm_65_6fb_description.urdf.xacro (robot description, xacro)
@@ -9,4 +9,9 @@
         link6_type:=$(arg link6_type)
     </xacro:include>
+    <link name="world"/>
+    <joint name="world_to_base" type="fixed">
+        <parent link="world"/>
+        <child link="base_link"/>
+    </joint>
     <!-- Import control_xacro -->
     <xacro:include filename="rm_65_description.ros2_control.xacro" />
